File: KiCad/TPS61092RSAR/TPS61092RSAR.kicad_pcb (KiCad board)
At the start: 2 copper layers, 8 parts, among them IC1 TPS61092RSAR

Commit message: Add files via upload
Parts:
- L1: footprint LQH44PH100MPRL -> INDPM4040X210N
- moved L1 0.51 mm to (180.2, 86.1)
